File: Schematic/Project1.kicad_sch (KiCad schematic)
At the start: 7 parts, among them J1 USB_C_Receptacle_USB2.0_14P, SW1 SW_Push, U1 ESP32-WROOM-32, U2 MAX7219, U3 AMS1117-3.3

Commit message: Add files via upload
Other:
- title: (none) -> Schematic
Changed lines of the file:
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@@
 	(generator_version "9.0")
 	(paper "A4")
+	(title_block
+		(title "Schematic")
+		(comment 1 "HO CHI MINH CITY UNIVERSITY OF TECHNOLOGY")
+	)
 	(junction
 		(at 245.11 120.65)
